File: Eagle/ALU/ALU.sch (EAGLE design)
At the start: 45 parts

Commit message: finished most boards
Parts:
- removed LED16: RED, led:LED3MM
- removed R15: 220, rcl:R-US_0204/7
- added C1, C2, C3, C4: (no value), rcl:C-US025-024X044
- added LED0: RED, led:LED3MM
- added R0: 220, rcl:R-US_0204/7
Connections:
- removed net N$89 (its old number): LED15.A, R15.1
- new net N$103: LED0.A, R0.1
- net N$52: now also C1.1, C2.1, C3.1, C4.1, LED0.C; no longer LED16.C
- net N$54: now also C1.2, C2.2, C3.2, C4.2
- net N$71: now also R0.2; no longer R1.2
- net N$73: now also R1.2; no longer R2.2
- net N$74: now also R2.2; no longer R3.2
- net N$75: now also R3.2; no longer R4.2
- net N$76: now also R4.2; no longer R5.2
- net N$77: now also R5.2; no longer R6.2
- net N$78: now also R6.2; no longer R7.2
- net N$79: now also R7.2; no longer R8.2
- net N$80: now also R8.2; no longer R9.2
- net N$81: now also R9.2; no longer R10.2
- net N$82: now also R10.2; no longer R11.2
- net N$83: now also R11.2; no longer R12.2
- net N$84: now also R12.2; no longer R13.2
- net N$85: now also R13.2; no longer R14.2
- net N$87: now also LED15.A; no longer LED16.A
- net N$88: now also R14.2; no longer R15.2
Other:
- moved on the sheet: LED1, LED10, LED11, LED12, LED13, LED14, LED15, LED2, LED3, LED4, LED5, LED6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
