File: Eagle/ALU/ALU.brd (EAGLE design)
At the start: 100 x 100 mm, 45 parts

Commit message: finished most boards
Parts:
- removed LED16: RED, led:LED3MM
- removed R15: 220, rcl:0204/7
- added C1, C2, C3, C4: (no value), rcl:C025-024X044
- added LED0: RED, led:LED3MM
- added R0: 220, rcl:0204/7
- added U$1, U$2, U$3, U$4: (no value), holes:2,8
- moved LED1 61.7 mm to (86.0, 76.0), turned to 90 degrees
- moved LED2 55.4 mm to (81.0, 76.0), turned to 90 degrees
- moved R1 52.7 mm to (86.0, 68.0), turned to 270 degrees
- moved LED15 50.4 mm to (16.0, 76.0), turned to 90 degrees
- moved LED3 49.2 mm to (76.0, 76.0), turned to 90 degrees
- moved R2 46.3 mm to (81.0, 68.0), turned to 270 degrees
- moved LED14 44.6 mm to (21.0, 76.0), turned to 90 degrees
- moved LED4 43.4 mm to (71.0, 76.0), turned to 90 degrees
- moved XOR_12-15 41.6 mm to (15.0, 28.2), turned to 90 degrees
- moved R16 40.5 mm to (16.0, 68.0), turned to 270 degrees
- moved R3 40.0 mm to (76.0, 68.0), turned to 270 degrees
- moved LED13 39.1 mm to (26.0, 76.0), turned to 90 degrees
- moved LED5 38.0 mm to (66.0, 76.0), turned to 90 degrees
- moved ADDER_4-7 35.0 mm to (49.9, 44.9), turned to 90 degrees
- moved LED12 34.1 mm to (31.0, 76.0), turned to 90 degrees
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Connections:
- removed net N$89 (its old number): LED15.A, R15.1
- new net N$103: LED0.A, R0.1
- net N$52: now also C1.1, C2.1, C3.1, C4.1, LED0.K; no longer LED16.K
- net N$54: now also C1.2, C2.2, C3.2, C4.2
- net N$71: now also R0.2; no longer R1.2
- net N$73: now also R1.2; no longer R2.2
- net N$74: now also R2.2; no longer R3.2
- net N$75: now also R3.2; no longer R4.2
- net N$76: now also R4.2; no longer R5.2
- net N$77: now also R5.2; no longer R6.2
- net N$78: now also R6.2; no longer R7.2
- net N$79: now also R7.2; no longer R8.2
- net N$80: now also R8.2; no longer R9.2
- net N$81: now also R9.2; no longer R10.2
- net N$82: now also R10.2; no longer R11.2
- net N$83: now also R11.2; no longer R12.2
- net N$84: now also R12.2; no longer R13.2
- net N$85: now also R13.2; no longer R14.2
- net N$87: now also LED15.A; no longer LED16.A
- net N$88: now also R14.2; no longer R15.2
Routing:
- net N$78: track 211.8 -> 81.6 mm, vias 1 -> 2
- net N$31: track 25.5 -> 113.5 mm
- net N$74: track 204.0 -> 123.0 mm
- net N$75: track 182.9 -> 106.4 mm, vias 0 -> 1
- net N$83: track 118.4 -> 190.2 mm
- net N$33: track 26.0 -> 90.4 mm, vias 0 -> 2
- net N$54: track 295.1 -> 233.6 mm, vias 1 -> 2
- net N$16: track 54.7 -> 115.8 mm, vias 1 -> 0
- net N$52: track 319.2 -> 376.9 mm, vias 1 -> 3
- net N$72: track 184.5 -> 237.9 mm, vias 0 -> 1
- net N$34: track 28.3 -> 78.7 mm
- net N$13: track 33.2 -> 81.7 mm, vias 0 -> 3
- net N$49: track 24.1 -> 68.2 mm
- net N$45: track 53.3 -> 94.7 mm
- net N$86: track 72.3 -> 113.7 mm, vias 3 -> 2
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
Commit message: added gerber files for each board
Other:
- board text added: "MARIE PC: ALU Architecture design by: Dr. Linda Null Hardware implementation by: Richard Bowser"
Changed lines of the file:
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@@
 <wire x1="100" y1="100" x2="0" y2="100" width="0" layer="20"/>
 <wire x1="0" y1="100" x2="0" y2="0" width="0" layer="20"/>
+<text x="62" y="86" size="1.778" layer="26" rot="MR0">MARIE PC:
+ALU
+Architecture design by: Dr. Linda Null
+Hardware implementation by: Richard Bowser</text>
 </plain>
 <attributes>
@@
 </drawing>
 <compatibility>
+<note version="6.3" minversion="6.2.2" severity="warning">
+Since Version 6.2.2 text objects can contain more than one line,
+which will not be processed correctly with this version.
+</note>
 <note version="8.2" severity="warning">
 Since Version 8.2, EAGLE supports online libraries. The ids
