File: Eagle/Program Counter/Program Counter.sch (EAGLE design)
At the start: 30 parts, among them J1 55959-2430

Commit message: Worked on IR
Connections:
- new net B12: BUFFER_8-11.Y5, J1.10
- new net B13: BUFFER_8-11.Y6, J1.12
- new net B14: BUFFER_8-11.Y7, J1.14
- new net B15: BUFFER_8-11.Y8, J1.16
- net GND: no longer BUFFER_8-11.Y5, BUFFER_8-11.Y6, BUFFER_8-11.Y7, BUFFER_8-11.Y8
Changed lines of the file:
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@@
 <junction x="-10.16" y="71.12"/>
 <wire x1="-10.16" y1="68.58" x2="-10.16" y2="60.96" width="0.1524" layer="91"/>
-<wire x1="-10.16" y1="60.96" x2="-43.18" y2="60.96" width="0.1524" layer="91"/>
 <junction x="-10.16" y="68.58"/>
-<pinref part="BUFFER_8-11" gate="G$1" pin="Y5"/>
-<wire x1="-40.64" y1="76.2" x2="-43.18" y2="76.2" width="0.1524" layer="91"/>
-<wire x1="-43.18" y1="76.2" x2="-43.18" y2="73.66" width="0.1524" layer="91"/>
-<pinref part="BUFFER_8-11" gate="G$1" pin="Y6"/>
-<wire x1="-43.18" y1="73.66" x2="-40.64" y2="73.66" width="0.1524" layer="91"/>
-<pinref part="BUFFER_8-11" gate="G$1" pin="Y7"/>
-<wire x1="-40.64" y1="71.12" x2="-43.18" y2="71.12" width="0.1524" layer="91"/>
-<wire x1="-43.18" y1="71.12" x2="-43.18" y2="73.66" width="0.1524" layer="91"/>
-<junction x="-43.18" y="73.66"/>
-<pinref part="BUFFER_8-11" gate="G$1" pin="Y8"/>
-<wire x1="-40.64" y1="68.58" x2="-43.18" y2="68.58" width="0.1524" layer="91"/>
-<wire x1="-43.18" y1="68.58" x2="-43.18" y2="71.12" width="0.1524" layer="91"/>
-<junction x="-43.18" y="71.12"/>
-<wire x1="-43.18" y1="60.96" x2="-43.18" y2="68.58" width="0.1524" layer="91"/>
-<junction x="-43.18" y="68.58"/>
 <wire x1="-10.16" y1="60.96" x2="2.54" y2="60.96" width="0.1524" layer="91"/>
 <wire x1="2.54" y1="60.96" x2="2.54" y2="5.08" width="0.1524" layer="91"/>
-<junction x="-10.16" y="60.96"/>
 <pinref part="BUFFER_0-8" gate="G$1" pin="GND"/>
 <wire x1="2.54" y1="5.08" x2="-10.16" y2="5.08" width="0.1524" layer="91"/>
@@
 </segment>
 </net>
+<net name="B12" class="0">
+<segment>
+<pinref part="J1" gate="G$1" pin="10"/>
+<wire x1="-152.4" y1="48.26" x2="-154.94" y2="48.26" width="0.1524" layer="91"/>
+<label x="-154.94" y="48.26" size="1.778" layer="95" rot="R180"/>
+</segment>
+<segment>
+<pinref part="BUFFER_8-11" gate="G$1" pin="Y5"/>
+<wire x1="-40.64" y1="76.2" x2="-43.18" y2="76.2" width="0.1524" layer="91"/>
+<label x="-43.18" y="76.2" size="1.778" layer="95" rot="R180"/>
+</segment>
+</net>
+<net name="B13" class="0">
+<segment>
+<pinref part="J1" gate="G$1" pin="12"/>
+<wire x1="-152.4" y1="45.72" x2="-154.94" y2="45.72" width="0.1524" layer="91"/>
+<label x="-154.94" y="45.72" size="1.778" layer="95" rot="R180"/>
+</segment>
+<segment>
+<pinref part="BUFFER_8-11" gate="G$1" pin="Y6"/>
+<wire x1="-40.64" y1="73.66" x2="-43.18" y2="73.66" width="0.1524" layer="91"/>
+<label x="-43.18" y="73.66" size="1.778" layer="95" rot="R180"/>
+</segment>
+</net>
+<net name="B14" class="0">
+<segment>
+<pinref part="J1" gate="G$1" pin="14"/>
+<wire x1="-152.4" y1="43.18" x2="-154.94" y2="43.18" width="0.1524" layer="91"/>
+<label x="-154.94" y="43.18" size="1.778" layer="95" rot="R180"/>
+</segment>
+<segment>
+<pinref part="BUFFER_8-11" gate="G$1" pin="Y7"/>
+<wire x1="-40.64" y1="71.12" x2="-43.18" y2="71.12" width="0.1524" layer="91"/>
+<label x="-43.18" y="71.12" size="1.778" layer="95" rot="R180"/>
+</segment>
+</net>
+<net name="B15" class="0">
+<segment>
+<pinref part="J1" gate="G$1" pin="16"/>
+<wire x1="-152.4" y1="40.64" x2="-154.94" y2="40.64" width="0.1524" layer="91"/>
+<label x="-154.94" y="40.64" size="1.778" layer="95" rot="R180"/>
+</segment>
+<segment>
+<pinref part="BUFFER_8-11" gate="G$1" pin="Y8"/>
+<wire x1="-40.64" y1="68.58" x2="-43.18" y2="68.58" width="0.1524" layer="91"/>
+<label x="-43.18" y="68.58" size="1.778" layer="95" rot="R180"/>
+</segment>
+</net>

Commit message: finished most boards
Parts:
- added C1, C2, C3, C4: (no value), rcl:C-US025-024X044
- renumbered J1 to BUS
Connections:
- net GND: now also C1.1, C2.1, C3.1, C4.1
- net VCC: now also C1.2, C2.2, C3.2, C4.2
