File: Eagle/Program Counter/Program Counter.brd (EAGLE design)
At the start: 100 x 100 mm, 30 parts, among them J1 55959-2430

Commit message: finished most boards
Parts:
- added C1, C2, C3, C4: (no value), rcl:C025-024X044
- added U$1, U$2, U$3, U$4: (no value), holes:2,8
- moved LED11 66.3 mm to (13.0, 87.0), turned to 90 degrees
- moved LED10 60.5 mm to (18.0, 87.0), turned to 90 degrees
- moved R11 58.6 mm to (13.0, 78.0), turned to 270 degrees
- moved LED9 55.1 mm to (23.0, 87.0), turned to 90 degrees
- moved R10 52.8 mm to (18.0, 78.0), turned to 270 degrees
- moved LED8 50.0 mm to (28.0, 87.0), turned to 90 degrees
- moved R9 47.2 mm to (23.0, 78.0), turned to 270 degrees
- moved LED7 45.5 mm to (33.0, 87.0), turned to 90 degrees
- moved LED0 43.2 mm to (68.0, 87.0), turned to 90 degrees
- moved LED6 41.8 mm to (38.0, 87.0), turned to 90 degrees
- moved R8 41.8 mm to (28.0, 78.0), turned to 270 degrees
- moved LED1 39.9 mm to (63.0, 87.0), turned to 90 degrees
- moved LED5 38.9 mm to (43.0, 87.0), turned to 90 degrees
- moved LED2 37.7 mm to (58.0, 87.0), turned to 90 degrees
- moved LED4 37.2 mm to (48.0, 87.0), turned to 90 degrees
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- renumbered J1 to BUS
Connections:
- net GND: now also C1.1, C2.1, C3.1, C4.1
- net VCC: now also C1.2, C2.2, C3.2, C4.2
Routing:
- net PC7: track 51.8 -> 151.7 mm, vias 0 -> 1
- net PCO: track 138.6 -> 86.2 mm
- net B5: track 132.6 -> 85.1 mm
- net PC3: track 71.2 -> 115.8 mm, vias 1 -> 0
- net PC5: track 81.1 -> 125.7 mm
- net PC4: track 89.8 -> 132.2 mm, vias 0 -> 1
- net CE: track 168.5 -> 207.3 mm, vias 0 -> 1
- net PC9: track 76.6 -> 114.5 mm, vias 0 -> 1
- net VCC: track 226.8 -> 261.2 mm, vias 0 -> 1
- net B15: track 0.00 -> 32.8 mm
- net B14: track 0.00 -> 32.6 mm
- net B13: track 0.00 -> 32.4 mm
- net PC8: track 76.0 -> 108.3 mm
- net PC2: track 79.5 -> 111.8 mm, vias 1 -> 0
- net B12: track 0.00 -> 32.2 mm
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
Commit message: added gerber files for each board
Other:
- board text added: "MARIE PC Program Counter Architecture design by: Dr. Linda Null Hardware implementation by: Richard Bowser"
Changed lines of the file:
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@@
 <wire x1="100" y1="100" x2="0" y2="100" width="0" layer="20"/>
 <wire x1="0" y1="100" x2="0" y2="0" width="0" layer="20"/>
+<text x="71" y="36" size="1.778" layer="26" rot="MR0">MARIE PC
+Program Counter
+Architecture design by: Dr. Linda Null
+Hardware implementation by: Richard Bowser</text>
 </plain>
 <attributes>
@@
 </drawing>
 <compatibility>
+<note version="6.3" minversion="6.2.2" severity="warning">
+Since Version 6.2.2 text objects can contain more than one line,
+which will not be processed correctly with this version.
+</note>
 <note version="8.2" severity="warning">
 Since Version 8.2, EAGLE supports online libraries. The ids

Commit message: started adding revision 2 to fix errors in first set of boards
Parts:
- LED0: value (none) -> YELLOW
Changed lines of the file:
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@@
 <drawing>
 <settings>
-<setting alwaysvectorfont="yes"/>
+<setting alwaysvectorfont="no"/>
 <setting verticaltext="up"/>
 </settings>
@@
 <attribute name="VALUE" x="19.651" y="88.905" size="1.27" layer="27" ratio="10" rot="R90"/>
 </element>
-<element name="LED0" library="led" library_urn="urn:adsk.eagle:library:259" package="LED3MM" package3d_urn="urn:adsk.eagle:package:15797/1" value="" x="68" y="87" smashed="yes" rot="R90">
+<element name="LED0" library="led" library_urn="urn:adsk.eagle:library:259" package="LED3MM" package3d_urn="urn:adsk.eagle:package:15797/1" value="YELLOW" x="68" y="87" smashed="yes" rot="R90">
 <attribute name="NAME" x="67.619" y="88.905" size="1.27" layer="25" ratio="10" rot="R90"/>
 <attribute name="POPULARITY" value="97" x="68" y="87" size="1.778" layer="27" rot="R90" display="off"/>
