File: Eagle/MBR/MBR.brd (EAGLE design)
At the start: 100 x 100 mm, 39 parts

Commit message: finished most boards
Parts:
- added C1, C2, C3, C4: (no value), rcl:C025-024X044
- added U$1, U$2, U$3, U$4: (no value), holes:2,8
- moved LED1 86.5 mm to (91.0, 18.0), turned to 270 degrees
- moved LED2 79.4 mm to (86.0, 18.0), turned to 270 degrees
- moved LED3 72.3 mm to (81.0, 18.0), turned to 270 degrees
- moved LED4 65.3 mm to (76.0, 18.0), turned to 270 degrees
- moved LED0 62.8 mm to (96.0, 18.0), turned to 270 degrees
- moved LED5 58.3 mm to (71.0, 18.0), turned to 270 degrees
- moved R1 58.1 mm to (91.0, 33.0), turned to 90 degrees
- moved R2 51.9 mm to (86.0, 33.0), turned to 90 degrees
- moved LED6 51.2 mm to (66.0, 18.0), turned to 270 degrees
- moved OUTPUT_0-7 49.0 mm to (40.2, 65.3)
- moved REGISTER_0-7 47.2 mm to (91.0, 58.4)
- moved REGISTER_8-15 47.0 mm to (74.2, 58.4)
- moved R0 45.9 mm to (96.0, 33.0), turned to 90 degrees
- moved R3 45.6 mm to (81.0, 33.0), turned to 90 degrees
- moved LED7 44.2 mm to (61.0, 18.0), turned to 270 degrees
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Connections:
- removed net N$19: BOARD_CONNECTOR.20, CLOCK_GATE.10, CLOCK_GATE.12, CLOCK_GATE.13, CLOCK_GATE.4, CLOCK_GATE.5, CLOCK_GATE.7, CLOCK_GATE.9, LED0.K, LED1.K, LED10.K, LED11.K, LED12.K, LED13.K, LED14.K, LED15.K, LED2.K, LED3.K, LED4.K, LED5.K, LED6.K, LED7.K, LED8.K, LED9.K, OUTPUT_0-7.10, OUTPUT_8-15.10, REGISTER_0-7.1, REGISTER_0-7.10, REGISTER_8-15.1, REGISTER_8-15.10
- removed net N$5: BOARD_CONNECTOR.19, CLOCK_GATE.14, OUTPUT_0-7.20, OUTPUT_8-15.20, REGISTER_0-7.20, REGISTER_8-15.20
- new net GND: BOARD_CONNECTOR.20, C1.1, C2.1, C3.1, C4.1, CLOCK_GATE.10, CLOCK_GATE.12, CLOCK_GATE.13, CLOCK_GATE.4, CLOCK_GATE.5, CLOCK_GATE.7, CLOCK_GATE.9, LED0.K, LED1.K, LED10.K, LED11.K, LED12.K, LED13.K, LED14.K, LED15.K, LED2.K, LED3.K, LED4.K, LED5.K, LED6.K, LED7.K, LED8.K, LED9.K, OUTPUT_0-7.10, OUTPUT_8-15.10, REGISTER_0-7.1, REGISTER_0-7.10, REGISTER_8-15.1, REGISTER_8-15.10
- new net VCC: BOARD_CONNECTOR.19, C1.2, C2.2, C3.2, C4.2, CLOCK_GATE.14, OUTPUT_0-7.20, OUTPUT_8-15.20, REGISTER_0-7.20, REGISTER_8-15.20
Routing:
- net GND: track 0.00 -> 353.9 mm, vias 0 -> 1
- net MBR13: track 0.00 -> 184.2 mm, vias 0 -> 5
- net MBR12: track 0.00 -> 181.3 mm, vias 0 -> 4
- net MBR9: track 0.00 -> 179.0 mm, vias 0 -> 3
- net VCC: track 0.00 -> 178.8 mm
- net MBR14: track 0.00 -> 174.4 mm, vias 0 -> 2
- net MBR11: track 0.00 -> 165.9 mm, vias 0 -> 2
- net MBR4: track 0.00 -> 159.1 mm, vias 0 -> 3
- net N$6: track 0.00 -> 156.0 mm
- net MBR6: track 0.00 -> 154.8 mm, vias 0 -> 4
- net MBR5: track 0.00 -> 153.7 mm, vias 0 -> 5
- net MBR1: track 0.00 -> 147.2 mm, vias 0 -> 3
- net MBR8: track 0.00 -> 146.6 mm
- net N$7: track 0.00 -> 143.0 mm, vias 0 -> 2
- net MBR3: track 0.00 -> 142.1 mm, vias 0 -> 4
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
Commit message: added gerber files for each board
Other:
- board text added: "MARIE PC MBR Architecture design by: Dr. Linda Null Hardware Implementation by: Richard Bowser"
Changed lines of the file:
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@@
 <wire x1="100" y1="100" x2="0" y2="100" width="0" layer="20"/>
 <wire x1="0" y1="100" x2="0" y2="0" width="0" layer="20"/>
+<text x="82" y="43" size="1.778" layer="26" rot="MR0">MARIE PC
+MBR
+Architecture design by: Dr. Linda Null
+Hardware Implementation by: Richard Bowser</text>
 </plain>
 <attributes>
@@
 </drawing>
 <compatibility>
+<note version="6.3" minversion="6.2.2" severity="warning">
+Since Version 6.2.2 text objects can contain more than one line,
+which will not be processed correctly with this version.
+</note>
 <note version="8.2" severity="warning">
 Since Version 8.2, EAGLE supports online libraries. The ids
