File: Eagle/Memory/MAR.sch (EAGLE design)
At the start: 43 parts, among them J1 55959-1830

Commit message: added Clock
Parts:
- renumbered J1 to BUS
Changed lines of the file:
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@@
 <part name="R0" library="rcl" library_urn="urn:adsk.eagle:library:334" deviceset="R-US_" device="0204/7" package3d_urn="urn:adsk.eagle:package:23498/2" value="220"/>
 <part name="DIP_8-11" library="SamacSys_Parts" deviceset="1825360-3" device=""/>
-<part name="J1" library="SamacSys_Parts" deviceset="55959-1830" device=""/>
+<part name="BUS" library="SamacSys_Parts" deviceset="55959-1830" device=""/>
 <part name="C1" library="rcl" library_urn="urn:adsk.eagle:library:334" deviceset="C-US" device="025-024X044" package3d_urn="urn:adsk.eagle:package:23630/1"/>
 <part name="C2" library="rcl" library_urn="urn:adsk.eagle:library:334" deviceset="C-US" device="025-024X044" package3d_urn="urn:adsk.eagle:package:23630/1"/>
@@
 <attribute name="VALUE" x="78.74" y="-87.63" size="1.778" layer="96" rot="R90" align="center-left"/>
 </instance>
-<instance part="J1" gate="G$1" x="193.04" y="35.56" smashed="yes">
+<instance part="BUS" gate="G$1" x="193.04" y="35.56" smashed="yes">
 <attribute name="NAME" x="212.09" y="43.18" size="1.778" layer="95" align="center-left"/>
 <attribute name="VALUE" x="212.09" y="40.64" size="1.778" layer="96" align="center-left"/>
@@
 </segment>
 <segment>
-<pinref part="J1" gate="G$1" pin="17"/>
+<pinref part="BUS" gate="G$1" pin="17"/>
 <wire x1="193.04" y1="15.24" x2="190.5" y2="15.24" width="0.1524" layer="91"/>
 <label x="190.5" y="15.24" size="1.778" layer="95" rot="R180"/>
@@
 <wire x1="193.04" y1="35.56" x2="190.5" y2="35.56" width="0.1524" layer="91"/>
 <label x="190.5" y="35.56" size="1.778" layer="95" rot="R180"/>
-<pinref part="J1" gate="G$1" pin="1"/>
+<pinref part="BUS" gate="G$1" pin="1"/>
 </segment>
 <segment>
@@
 <wire x1="193.04" y1="33.02" x2="190.5" y2="33.02" width="0.1524" layer="91"/>
 <label x="190.5" y="33.02" size="1.778" layer="95" rot="R180"/>
-<pinref part="J1" gate="G$1" pin="3"/>
+<pinref part="BUS" gate="G$1" pin="3"/>
 </segment>
 <segment>
@@
 <wire x1="193.04" y1="30.48" x2="190.5" y2="30.48" width="0.1524" layer="91"/>
 <label x="190.5" y="30.48" size="1.778" layer="95" rot="R180"/>
-<pinref part="J1" gate="G$1" pin="5"/>
+<pinref part="BUS" gate="G$1" pin="5"/>
 </segment>
 <segment>
@@
 <wire x1="193.04" y1="27.94" x2="190.5" y2="27.94" width="0.1524" layer="91"/>
 <label x="190.5" y="27.94" size="1.778" layer="95" rot="R180"/>
-<pinref part="J1" gate="G$1" pin="7"/>
+<pinref part="BUS" gate="G$1" pin="7"/>
 </segment>
 <segment>
@@
 <wire x1="193.04" y1="25.4" x2="190.5" y2="25.4" width="0.1524" layer="91"/>
 <label x="190.5" y="25.4" size="1.778" layer="95" rot="R180"/>
-<pinref part="J1" gate="G$1" pin="9"/>
+<pinref part="BUS" gate="G$1" pin="9"/>
 </segment>
 <segment>
@@
 <wire x1="193.04" y1="22.86" x2="190.5" y2="22.86" width="0.1524" layer="91"/>
 <label x="190.5" y="22.86" size="1.778" layer="95" rot="R180"/>
-<pinref part="J1" gate="G$1" pin="11"/>
+<pinref part="BUS" gate="G$1" pin="11"/>
 </segment>
 <segment>
@@
 <wire x1="193.04" y1="20.32" x2="190.5" y2="20.32" width="0.1524" layer="91"/>
 <label x="190.5" y="20.32" size="1.778" layer="95" rot="R180"/>
-<pinref part="J1" gate="G$1" pin="13"/>
+<pinref part="BUS" gate="G$1" pin="13"/>
 </segment>
 </net>
@@
 <wire x1="193.04" y1="17.78" x2="190.5" y2="17.78" width="0.1524" layer="91"/>
 <label x="190.5" y="17.78" size="1.778" layer="95" rot="R180"/>
-<pinref part="J1" gate="G$1" pin="15"/>
+<pinref part="BUS" gate="G$1" pin="15"/>
 </segment>
 </net>
@@
 <wire x1="215.9" y1="35.56" x2="218.44" y2="35.56" width="0.1524" layer="91"/>
 <label x="218.44" y="35.56" size="1.778" layer="95"/>
-<pinref part="J1" gate="G$1" pin="2"/>
+<pinref part="BUS" gate="G$1" pin="2"/>
 </segment>
 </net>
@@
 <wire x1="215.9" y1="33.02" x2="218.44" y2="33.02" width="0.1524" layer="91"/>
 <label x="218.44" y="33.02" size="1.778" layer="95"/>
-<pinref part="J1" gate="G$1" pin="4"/>
+<pinref part="BUS" gate="G$1" pin="4"/>
 </segment>
 </net>
@@
 <wire x1="215.9" y1="30.48" x2="218.44" y2="30.48" width="0.1524" layer="91"/>
 <label x="218.44" y="30.48" size="1.778" layer="95"/>
-<pinref part="J1" gate="G$1" pin="6"/>
+<pinref part="BUS" gate="G$1" pin="6"/>
 </segment>
 </net>
@@
 <wire x1="215.9" y1="27.94" x2="218.44" y2="27.94" width="0.1524" layer="91"/>
 <label x="218.44" y="27.94" size="1.778" layer="95"/>
-<pinref part="J1" gate="G$1" pin="8"/>
+<pinref part="BUS" gate="G$1" pin="8"/>
 </segment>
 </net>
@@
 <wire x1="215.9" y1="20.32" x2="218.44" y2="20.32" width="0.1524" layer="91"/>
 <label x="218.44" y="20.32" size="1.778" layer="95"/>
-<pinref part="J1" gate="G$1" pin="14"/>
+<pinref part="BUS" gate="G$1" pin="14"/>
 </segment>
 <segment>
@@
 <wire x1="215.9" y1="25.4" x2="218.44" y2="25.4" width="0.1524" layer="91"/>
 <label x="218.44" y="25.4" size="1.778" layer="95"/>
-<pinref part="J1" gate="G$1" pin="10"/>
+<pinref part="BUS" gate="G$1" pin="10"/>
 </segment>
 </net>
@@
 <wire x1="215.9" y1="22.86" x2="218.44" y2="22.86" width="0.1524" layer="91"/>
 <label x="218.44" y="22.86" size="1.778" layer="95"/>
-<pinref part="J1" gate="G$1" pin="12"/>
+<pinref part="BUS" gate="G$1" pin="12"/>
 </segment>
 <segment>
@@
 <wire x1="215.9" y1="17.78" x2="218.44" y2="17.78" width="0.1524" layer="91"/>
 <label x="218.44" y="17.78" size="1.778" layer="95"/>
-<pinref part="J1" gate="G$1" pin="16"/>
-</segment>
-<segment>
+<pinref part="BUS" gate="G$1" pin="16"/>
+</segment>
+<segment>

Commit message: added gerber files for each board
Parts:
- added LEDPRGM: RED, led:LED3MM
- added LEDRUN: GREEN, led:LED3MM
- added RPRGM, RRUN: 220, rcl:R-US_0204/7
Connections:
- new net N$12: LEDPRGM.A, RPRGM.1
- new net N$13: LEDRUN.A, RRUN.1
- new net N$14: PRGM_SWITCH.1, RRUN.2
- net GND: now also LEDPRGM.C, LEDRUN.C
- net PRGM: now also RPRGM.2
Changed lines of the file:
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@@
 <part name="C3" library="rcl" library_urn="urn:adsk.eagle:library:334" deviceset="C-US" device="025-024X044" package3d_urn="urn:adsk.eagle:package:23630/1"/>
 <part name="C4" library="rcl" library_urn="urn:adsk.eagle:library:334" deviceset="C-US" device="025-024X044" package3d_urn="urn:adsk.eagle:package:23630/1"/>
+<part name="LEDPRGM" library="led" library_urn="urn:adsk.eagle:library:259" deviceset="LED" device="3MM" package3d_urn="urn:adsk.eagle:package:15797/1" value="RED"/>
+<part name="LEDRUN" library="led" library_urn="urn:adsk.eagle:library:259" deviceset="LED" device="3MM" package3d_urn="urn:adsk.eagle:package:15797/1" value="GREEN"/>
+<part name="RPRGM" library="rcl" library_urn="urn:adsk.eagle:library:334" deviceset="R-US_" device="0204/7" package3d_urn="urn:adsk.eagle:package:23498/2" value="220"/>
+<part name="RRUN" library="rcl" library_urn="urn:adsk.eagle:library:334" deviceset="R-US_" device="0204/7" package3d_urn="urn:adsk.eagle:package:23498/2" value="220"/>
 </parts>
 <sheets>
@@
 <attribute name="VALUE" x="242.824" y="-13.589" size="1.778" layer="96" rot="R180"/>
 </instance>
+<instance part="LEDPRGM" gate="G$1" x="149.86" y="-149.86" smashed="yes">
+<attribute name="NAME" x="153.416" y="-154.432" size="1.778" layer="95" rot="R90"/>
+<attribute name="VALUE" x="155.575" y="-154.432" size="1.778" layer="96" rot="R90"/>
+</instance>
+<instance part="LEDRUN" gate="G$1" x="167.64" y="-149.86" smashed="yes">
+<attribute name="NAME" x="171.196" y="-154.432" size="1.778" layer="95" rot="R90"/>
+<attribute name="VALUE" x="173.355" y="-154.432" size="1.778" layer="96" rot="R90"/>
+</instance>
+<instance part="RPRGM" gate="G$1" x="149.86" y="-142.24" smashed="yes" rot="R90">
+<attribute name="NAME" x="148.3614" y="-146.05" size="1.778" layer="95" rot="R90"/>
+<attribute name="VALUE" x="153.162" y="-146.05" size="1.778" layer="96" rot="R90"/>
+</instance>
+<instance part="RRUN" gate="G$1" x="167.64" y="-142.24" smashed="yes" rot="R90">
+<attribute name="NAME" x="166.1414" y="-146.05" size="1.778" layer="95" rot="R90"/>
+<attribute name="VALUE" x="170.942" y="-146.05" size="1.778" layer="96" rot="R90"/>
+</instance>
 </instances>
 <busses>
@@
 <wire x1="193.04" y1="15.24" x2="190.5" y2="15.24" width="0.1524" layer="91"/>
 <label x="190.5" y="15.24" size="1.778" layer="95" rot="R180"/>
+</segment>
+<segment>
+<pinref part="RPRGM" gate="G$1" pin="2"/>
+<wire x1="149.86" y1="-137.16" x2="149.86" y2="-134.62" width="0.1524" layer="91"/>
+<label x="149.86" y="-134.62" size="1.778" layer="95" rot="R90"/>
 </segment>
 </net>
@@
 <junction x="116.84" y="-160.02"/>
 <label x="121.92" y="-160.02" size="1.778" layer="95"/>
+<wire x1="116.84" y1="-160.02" x2="116.84" y2="-167.64" width="0.1524" layer="91"/>
+<pinref part="LEDPRGM" gate="G$1" pin="C"/>
+<wire x1="149.86" y1="-154.94" x2="149.86" y2="-157.48" width="0.1524" layer="91"/>
+<wire x1="149.86" y1="-157.48" x2="167.64" y2="-157.48" width="0.1524" layer="91"/>
+<pinref part="LEDRUN" gate="G$1" pin="C"/>
+<wire x1="167.64" y1="-157.48" x2="167.64" y2="-154.94" width="0.1524" layer="91"/>
+<wire x1="116.84" y1="-167.64" x2="149.86" y2="-167.64" width="0.1524" layer="91"/>
+<wire x1="149.86" y1="-167.64" x2="149.86" y2="-157.48" width="0.1524" layer="91"/>
+<junction x="149.86" y="-157.48"/>
 </segment>
 <segment>
@@
 </segment>
 </net>
+<net name="N$12" class="0">
+<segment>
+<pinref part="LEDPRGM" gate="G$1" pin="A"/>
+<pinref part="RPRGM" gate="G$1" pin="1"/>
+</segment>
+</net>
+<net name="N$13" class="0">
+<segment>
+<pinref part="LEDRUN" gate="G$1" pin="A"/>
+<pinref part="RRUN" gate="G$1" pin="1"/>
+</segment>
+</net>
+<net name="N$14" class="0">
+<segment>
+<pinref part="RRUN" gate="G$1" pin="2"/>
+<pinref part="PRGM_SWITCH" gate="G$1" pin="1"/>
+<wire x1="167.64" y1="-137.16" x2="167.64" y2="-55.88" width="0.1524" layer="91"/>
+<wire x1="167.64" y1="-55.88" x2="182.88" y2="-55.88" width="0.1524" layer="91"/>
+</segment>
+</net>
