File: Eagle/Memory/MAR.brd (EAGLE design)
At the start: 160 x 100 mm, 39 parts, among them J1 55959-1830

Commit message: finished most boards
Parts:
- added C1, C2, C3, C4: (no value), rcl:C025-024X044
Connections:
- net GND: now also C1.1, C2.1, C3.1, C4.1
- net VCC: now also C1.2, C2.2, C3.2, C4.2

Commit message: added Clock
Parts:
- removed J1: 55959-1830, SamacSys_Parts:SHDR18W65P250X200_2X9_2140X140
- added BUS: 55959-1830, SamacSys_Parts:SHDR18W65P250X200_2X9_2140X140
- added U$1, U$2, U$3, U$4: (no value), holes:2,8
- moved C1 183.9 mm to (91.4, 38.2)
- moved C2 183.9 mm to (91.4, 33.1)
- moved C3 183.9 mm to (91.4, 28.0)
- moved C4 183.9 mm to (91.4, 22.9)
- moved LED3 158.9 mm to (62.3, 24.8), turned to 270 degrees
- moved R4 153.8 mm to (57.9, 34.2), turned to 270 degrees
- moved LED2 151.8 mm to (67.5, 24.9), turned to 270 degrees
- moved R3 148.7 mm to (62.6, 34.3), turned to 270 degrees
- moved LED1 144.7 mm to (72.5, 24.9), turned to 270 degrees
- moved R2 143.8 mm to (67.3, 34.1), turned to 270 degrees
- moved R1 139.5 mm to (72.6, 34.1), turned to 270 degrees
- moved LED0 137.5 mm to (77.5, 24.9), turned to 270 degrees
- moved LED9 136.4 mm to (33.4, 24.9), turned to 270 degrees
- moved R0 135.1 mm to (78.1, 34.3), turned to 270 degrees
- moved DIP_0-7 131.4 mm to (76.7, 7.95), turned to 90 degrees
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Connections:
- net B0: now also BUS.1; no longer J1.1
- net B1: now also BUS.3; no longer J1.3
- net B10: now also BUS.6; no longer J1.6
- net B11: now also BUS.8; no longer J1.8
- net B2: now also BUS.5; no longer J1.5
- net B3: now also BUS.7; no longer J1.7
- net B4: now also BUS.9; no longer J1.9
- net B5: now also BUS.11; no longer J1.11
- net B6: now also BUS.13; no longer J1.13
- net B7: now also BUS.15; no longer J1.15
- net B8: now also BUS.2; no longer J1.2
- net B9: now also BUS.4; no longer J1.4
- net CLK: now also BUS.14; no longer J1.14
- net GND: now also BUS.16; no longer J1.16
- net MARI: now also BUS.10; no longer J1.10
- net PRGM: now also BUS.17; no longer J1.17
- net VCC: now also BUS.12; no longer J1.12
Routing:
- net GND: track 0.00 -> 449.4 mm, vias 0 -> 1
- net VCC: track 0.00 -> 294.4 mm, vias 0 -> 3
- net A0: track 0.00 -> 223.8 mm
- net PRGM: track 0.00 -> 223.2 mm, vias 0 -> 2
- net A3: track 0.00 -> 184.3 mm, vias 0 -> 2
- net A2: track 0.00 -> 177.1 mm, vias 0 -> 3
- net B2: track 0.00 -> 172.6 mm, vias 0 -> 1
- net A4: track 0.00 -> 163.0 mm, vias 0 -> 1
- net B3: track 0.00 -> 162.5 mm, vias 0 -> 1
- net A10: track 0.00 -> 150.6 mm, vias 0 -> 2
- net R1: track 0.00 -> 150.1 mm
- net A6: track 0.00 -> 139.3 mm, vias 0 -> 4
- net B7: track 0.00 -> 136.7 mm, vias 0 -> 2
- net B11: track 0.00 -> 135.0 mm, vias 0 -> 1
- net B6: track 0.00 -> 134.4 mm, vias 0 -> 3
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Other:
- board size 160 x 100 mm -> 100 x 100 mm

Commit message: added gerber files for each board
Parts:
- added LEDPRGM: RED, led:LED3MM
- added LEDRUN: GREEN, led:LED3MM
- added RPRGM, RRUN: 220, rcl:0204/7
Connections:
- new net N$12: LEDPRGM.A, RPRGM.1
- new net N$13: LEDRUN.A, RRUN.1
- new net N$14: PRGM_SWITCH.1, RRUN.2
- net GND: now also LEDPRGM.K, LEDRUN.K
- net PRGM: now also RPRGM.2
Routing:
- net A1: track 131.2 -> 223.2 mm
- net A5: track 124.7 -> 203.5 mm
- net PRGM: track 223.2 -> 295.9 mm, vias 2 -> 1
- net A7: track 103.3 -> 156.0 mm, vias 4 -> 3
- net A10: track 150.6 -> 100.3 mm, vias 2 -> 4
- net B11: track 135.0 -> 91.9 mm, vias 1 -> 2
- net B5: track 102.6 -> 145.5 mm, vias 3 -> 5
- net N$1: track 116.1 -> 75.7 mm, vias 0 -> 4
- net A6: track 139.3 -> 101.1 mm
- net GND: track 449.4 -> 486.9 mm
- net VCC: track 294.4 -> 328.5 mm, vias 3 -> 4
- net A11: track 83.8 -> 113.3 mm, vias 5 -> 1
- net R2: track 60.3 -> 87.6 mm
- net A2: track 177.1 -> 150.4 mm, vias 3 -> 6
- net B4: track 89.9 -> 112.3 mm
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Other:
- board text added: "MARIE PC MAR Architecture designed by: Dr. Linda Null Hardware implementation by: Richard Bowser"

Commit message: added gerber files for ordering boards
Other:
- board text added: "MARIE PC: MAR Architecture design by: Dr. Linda Null Hardware implementation by: Richard Bowser"
Changed lines of the file:
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@@
 <drawing>
 <settings>
-<setting alwaysvectorfont="yes"/>
+<setting alwaysvectorfont="no"/>
 <setting verticaltext="up"/>
 </settings>
@@
 Architecture designed by: Dr. Linda Null
 Hardware implementation by: Richard Bowser</text>
+<text x="72" y="40" size="1.778" layer="26" rot="MR0">MARIE PC:
+MAR
+Architecture design by: Dr. Linda Null
+Hardware implementation by: Richard Bowser</text>
 </plain>
