File: Eagle/Memory/memory.sch (EAGLE design)
At the start: 4 parts, among them IC1 AS6C6264-55PIN, IC2 AS6C6264-55PIN, J1 55959-1630, J2 55959-2030

Commit message: almost finished memory
Parts:
- removed IC1, IC2: AS6C6264-55PIN, SamacSys_Parts:AS6C6264-55PIN
- removed J1: 55959-1630, SamacSys_Parts:55959-1630
- removed J2: 55959-2030, SamacSys_Parts:55959-2030
- added AND_GATE: SN74HC08N, SamacSys_Parts:SN74HC08N
- added ARD/BRD_0-3, ARD/BRD_12-15, ARD/BRD_4-7, ARD/BRD_8-11, ARDUINO_WRITE, BOARD_WRITE, BUS/DIP_0-3, BUS/DIP_12-15, BUS/DIP_4-7, BUS/DIP_8-11: SN74HC157N, SamacSys_Parts:SN74HC157N
- added ARDUINO: 55959-1830, SamacSys_Parts:55959-1830
- added BUS: 55959-2430, SamacSys_Parts:55959-2430
- added DIP_0-7, DIP_8-15: ADE08A04, SamacSys_Parts:ADE08A04
- added MAR: 55959-1430, SamacSys_Parts:55959-1430
- added MEMORY_0-7, MEMORY_8-15: AS6C6264-55PIN, SamacSys_Parts:AS6C6264-55PIN
- added RAM_OUT_0-7, RAM_OUT_8-15: SN74HC541N, SamacSys_Parts:SN74HC541N
Connections:
- new net A0: MAR.1, MEMORY_0-7.A0, MEMORY_8-15.A0
- new net A1: MAR.2, MEMORY_0-7.A1, MEMORY_8-15.A1
- new net A10: MAR.12, MEMORY_0-7.A10, MEMORY_8-15.A10
- new net A11: MAR.13, MEMORY_0-7.A11, MEMORY_8-15.A11
- new net A2: MAR.3, MEMORY_0-7.A2, MEMORY_8-15.A2
- new net A3: MAR.4, MEMORY_0-7.A3, MEMORY_8-15.A3
- new net A4: MAR.5, MEMORY_0-7.A4, MEMORY_8-15.A4
- new net A5: MAR.6, MEMORY_0-7.A5, MEMORY_8-15.A5
- new net A6: MAR.8, MEMORY_0-7.A6, MEMORY_8-15.A6
- new net A7: MAR.9, MEMORY_0-7.A7, MEMORY_8-15.A7
- new net A8: MAR.10, MEMORY_0-7.A8, MEMORY_8-15.A8
- new net A9: MAR.11, MEMORY_0-7.A9, MEMORY_8-15.A9
- new net ARD0: ARD/BRD_0-3.1B, ARDUINO.1
- new net ARD1: ARD/BRD_0-3.2B, ARDUINO.3
- new net ARD10: ARD/BRD_8-11.3B, ARDUINO.6
- new net ARD11: ARD/BRD_8-11.4B, ARDUINO.8
- new net ARD12: ARD/BRD_12-15.1B, ARDUINO.10
- new net ARD13: ARD/BRD_12-15.2B, ARDUINO.12
- new net ARD14: ARD/BRD_12-15.3B, ARDUINO.14
- new net ARD15: ARD/BRD_12-15.4B, ARDUINO.16
- new net ARD2: ARD/BRD_0-3.3B, ARDUINO.5
- new net ARD3: ARD/BRD_0-3.4B, ARDUINO.7
- new net ARD4: ARD/BRD_4-7.1B, ARDUINO.9
- new net ARD5: ARD/BRD_4-7.2B, ARDUINO.11
- new net ARD6: ARD/BRD_4-7.3B, ARDUINO.13
- new net ARD7: ARD/BRD_4-7.4B, ARDUINO.15
- new net ARD8: ARD/BRD_8-11.1B, ARDUINO.2
- new net ARD9: ARD/BRD_8-11.2B, ARDUINO.4
- new net ARDPRGM: AND_GATE.1B, ARDUINO.18, ARDUINO_WRITE.!A!/B
- new net ARDWRITE: ARDUINO.17, ARDUINO_WRITE.1B
- new net B0: BUS.1, BUS/DIP_0-3.1A, RAM_OUT_0-7.Y1
- new net B1: BUS.3, BUS/DIP_0-3.2A, RAM_OUT_0-7.Y2
- new net B10: BUS.6, BUS/DIP_8-11.3A, RAM_OUT_8-15.Y3
- new net B11: BUS.8, BUS/DIP_8-11.4A, RAM_OUT_8-15.Y4
- new net B12: BUS.10, BUS/DIP_12-15.1A, RAM_OUT_8-15.Y5
- new net B13: BUS.12, BUS/DIP_12-15.2A, RAM_OUT_8-15.Y6
- new net B14: BUS.14, BUS/DIP_12-15.3A, RAM_OUT_8-15.Y7
- new net B15: BUS.16, BUS/DIP_12-15.4A, RAM_OUT_8-15.Y8
- new net B2: BUS.5, BUS/DIP_0-3.3A, RAM_OUT_0-7.Y3
- new net B3: BUS.7, BUS/DIP_0-3.4A, RAM_OUT_0-7.Y4
- new net B4: BUS.9, BUS/DIP_4-7.1A, RAM_OUT_0-7.Y5
- new net B5: BUS.11, BUS/DIP_4-7.2A, RAM_OUT_0-7.Y6
- new net B6: BUS.13, BUS/DIP_4-7.3A, RAM_OUT_0-7.Y7
- new net B7: BUS.15, BUS/DIP_4-7.4A, RAM_OUT_0-7.Y8
- new net B8: BUS.2, BUS/DIP_8-11.1A, RAM_OUT_8-15.Y1
- new net B9: BUS.4, BUS/DIP_8-11.2A, RAM_OUT_8-15.Y2
- new net BRD0: ARD/BRD_0-3.1A, BUS/DIP_0-3.1Y
- new net BRD1: ARD/BRD_0-3.2A, BUS/DIP_0-3.2Y
- new net BRD10: ARD/BRD_8-11.3A, BUS/DIP_8-11.3Y
- new net BRD11: ARD/BRD_8-11.4A, BUS/DIP_8-11.4Y
- new net BRD12: ARD/BRD_12-15.1A, BUS/DIP_12-15.1Y
- new net BRD13: ARD/BRD_12-15.2A, BUS/DIP_12-15.2Y
- new net BRD14: ARD/BRD_12-15.3A, BUS/DIP_12-15.3Y
- new net BRD15: ARD/BRD_12-15.4A, BUS/DIP_12-15.4Y
- new net BRD2: ARD/BRD_0-3.3A, BUS/DIP_0-3.3Y
- new net BRD3: ARD/BRD_0-3.4A, BUS/DIP_0-3.4Y
- new net BRD4: ARD/BRD_4-7.1A, BUS/DIP_4-7.1Y
- new net BRD5: ARD/BRD_4-7.2A, BUS/DIP_4-7.2Y
- new net BRD6: ARD/BRD_4-7.3A, BUS/DIP_4-7.3Y
- new net BRD7: ARD/BRD_4-7.4A, BUS/DIP_4-7.4Y
- new net BRD8: ARD/BRD_8-11.1A, BUS/DIP_8-11.1Y
- new net BRD9: ARD/BRD_8-11.2A, BUS/DIP_8-11.2Y
- new net CLK: AND_GATE.2A, BUS.21
- new net DIP0: BUS/DIP_0-3.1B, DIP_0-7.9
- new net DIP1: BUS/DIP_0-3.2B, DIP_0-7.10
- new net DIP10: BUS/DIP_8-11.3B, DIP_8-15.11
- new net DIP11: BUS/DIP_8-11.4B, DIP_8-15.12
- new net DIP12: BUS/DIP_12-15.1B, DIP_8-15.13
- new net DIP13: BUS/DIP_12-15.2B, DIP_8-15.14
- new net DIP14: BUS/DIP_12-15.3B, DIP_8-15.15
- new net DIP15: BUS/DIP_12-15.4B, DIP_8-15.16
- new net DIP2: BUS/DIP_0-3.3B, DIP_0-7.11
- new net DIP3: BUS/DIP_0-3.4B, DIP_0-7.12
- new net DIP4: BUS/DIP_4-7.1B, DIP_0-7.13
- new net DIP5: BUS/DIP_4-7.2B, DIP_0-7.14
- new net DIP6: BUS/DIP_4-7.3B, DIP_0-7.15
- new net DIP7: BUS/DIP_4-7.4B, DIP_0-7.16
- new net DIP8: BUS/DIP_8-11.1B, DIP_8-15.9
- new net DIP9: BUS/DIP_8-11.2B, DIP_8-15.10
- new net GND: AND_GATE.3A, AND_GATE.3B, AND_GATE.4A, AND_GATE.4B, AND_GATE.GND, ARD/BRD_0-3.!G, ARD/BRD_0-3.GND, ARD/BRD_12-15.!G, ARD/BRD_12-15.GND, ARD/BRD_4-7.!G, ARD/BRD_4-7.GND, ARD/BRD_8-11.!G, ARD/BRD_8-11.GND, ARDUINO_WRITE.!G, ARDUINO_WRITE.2A, ARDUINO_WRITE.2B, ARDUINO_WRITE.3A, ARDUINO_WRITE.3B, ARDUINO_WRITE.4A, ARDUINO_WRITE.4B, ARDUINO_WRITE.GND, BOARD_WRITE.!G, BOARD_WRITE.2A, BOARD_WRITE.2B, BOARD_WRITE.3A, BOARD_WRITE.3B, BOARD_WRITE.4A, BOARD_WRITE.4B, BOARD_WRITE.GND, BUS.20, BUS/DIP_0-3.!G, BUS/DIP_0-3.GND, BUS/DIP_12-15.!G, BUS/DIP_12-15.GND, BUS/DIP_4-7.!G, BUS/DIP_4-7.GND, BUS/DIP_8-11.!G, BUS/DIP_8-11.GND, MEMORY_0-7.A12, MEMORY_0-7.CE#, MEMORY_0-7.VSS, MEMORY_8-15.A12, MEMORY_8-15.CE#, MEMORY_8-15.VSS, RAM_OUT_0-7.GND, RAM_OUT_8-15.GND
- new net N$1: ARDUINO_WRITE.1Y, MEMORY_0-7.WE#, MEMORY_8-15.WE#
- new net N$2: BOARD_WRITE.1B
- new net N$3: ARDUINO_WRITE.1A, BOARD_WRITE.1Y
- new net PRGM: AND_GATE.1A, BOARD_WRITE.!A!/B, BUS/DIP_0-3.!A!/B, BUS/DIP_12-15.!A!/B, BUS/DIP_4-7.!A!/B, BUS/DIP_8-11.!A!/B, MAR.7
- new net RAM0: ARD/BRD_0-3.1Y, MEMORY_0-7.DQ0, RAM_OUT_0-7.A1
- new net RAM1: ARD/BRD_0-3.2Y, MEMORY_0-7.DQ1, RAM_OUT_0-7.A2
- new net RAM10: ARD/BRD_8-11.3Y, MEMORY_8-15.DQ2, RAM_OUT_8-15.A3
- new net RAM11: ARD/BRD_8-11.4Y, MEMORY_8-15.DQ3, RAM_OUT_8-15.A4
- new net RAM12: ARD/BRD_12-15.1Y, MEMORY_8-15.DQ4, RAM_OUT_8-15.A5
- new net RAM13: ARD/BRD_12-15.2Y, MEMORY_8-15.DQ5, RAM_OUT_8-15.A6
- new net RAM14: ARD/BRD_12-15.3Y, MEMORY_8-15.DQ6, RAM_OUT_8-15.A7
- new net RAM15: ARD/BRD_12-15.4Y, MEMORY_8-15.DQ7, RAM_OUT_8-15.A8
- new net RAM2: ARD/BRD_0-3.3Y, MEMORY_0-7.DQ2, RAM_OUT_0-7.A3
- new net RAM3: ARD/BRD_0-3.4Y, MEMORY_0-7.DQ3, RAM_OUT_0-7.A4
- new net RAM4: ARD/BRD_4-7.1Y, MEMORY_0-7.DQ4, RAM_OUT_0-7.A5
- new net RAM5: ARD/BRD_4-7.2Y, MEMORY_0-7.DQ5, RAM_OUT_0-7.A6
- new net RAM6: ARD/BRD_4-7.3Y, MEMORY_0-7.DQ6, RAM_OUT_0-7.A7
- new net RAM7: ARD/BRD_4-7.4Y, MEMORY_0-7.DQ7, RAM_OUT_0-7.A8
- new net RAM8: ARD/BRD_8-11.1Y, MEMORY_8-15.DQ0, RAM_OUT_8-15.A1
- new net RAM9: ARD/BRD_8-11.2Y, MEMORY_8-15.DQ1, RAM_OUT_8-15.A2
- new net RAMCLK: AND_GATE.2Y, BOARD_WRITE.1A
- new net RAMPROG: AND_GATE.1Y, ARD/BRD_0-3.!A!/B, ARD/BRD_12-15.!A!/B, ARD/BRD_4-7.!A!/B, ARD/BRD_8-11.!A!/B
- new net RI: AND_GATE.2B, BUS.18
- new net RO: BUS.17, MEMORY_0-7.OE#, MEMORY_8-15.OE#, RAM_OUT_0-7.!OE1, RAM_OUT_0-7.!OE2, RAM_OUT_8-15.!OE1, RAM_OUT_8-15.!OE2
- new net VCC: AND_GATE.VCC, ARD/BRD_0-3.VCC, ARD/BRD_12-15.VCC, ARD/BRD_4-7.VCC, ARD/BRD_8-11.VCC, ARDUINO_WRITE.VCC, BOARD_WRITE.VCC, BUS.19, BUS/DIP_0-3.VCC, BUS/DIP_12-15.VCC, BUS/DIP_4-7.VCC, BUS/DIP_8-11.VCC, DIP_0-7.1, DIP_0-7.2, DIP_0-7.3, DIP_0-7.4, DIP_0-7.5, DIP_0-7.6, DIP_0-7.7, DIP_0-7.8, DIP_8-15.1, DIP_8-15.2, DIP_8-15.3, DIP_8-15.4, DIP_8-15.5, DIP_8-15.6, DIP_8-15.7, DIP_8-15.8, MEMORY_0-7.CE2, MEMORY_0-7.VCC, MEMORY_8-15.CE2, MEMORY_8-15.VCC, RAM_OUT_0-7.VCC, RAM_OUT_8-15.VCC

Commit message: added parts needed to finish boards
Parts:
- added IC1: SN74HC02N, SamacSys_Parts:SN74HC02N
- added S1: MHPS2273N, SamacSys_Parts:MHPS2273N
Connections:
- net GND: now also S1.N.O._1
- net N$2: now also S1.COM_1
- net VCC: now also S1.N.C._1
Changed lines of the file:
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@@
 <part name="RAM_OUT_8-15" library="SamacSys_Parts" deviceset="SN74HC541N" device=""/>
 <part name="RAM_OUT_0-7" library="SamacSys_Parts" deviceset="SN74HC541N" device=""/>
+<part name="S1" library="SamacSys_Parts" deviceset="MHPS2273N" device=""/>
+<part name="IC1" library="SamacSys_Parts" deviceset="SN74HC02N" device=""/>
 </parts>
 <sheets>
@@
 <attribute name="NAME" x="181.61" y="185.42" size="1.778" layer="95" align="center-left"/>
 <attribute name="VALUE" x="181.61" y="182.88" size="1.778" layer="96" align="center-left"/>
+</instance>
+<instance part="S1" gate="G$1" x="236.22" y="-43.18" smashed="yes">
+<attribute name="NAME" x="265.43" y="-35.56" size="1.778" layer="95" align="center-left"/>
+<attribute name="VALUE" x="265.43" y="-38.1" size="1.778" layer="96" align="center-left"/>
+</instance>
+<instance part="IC1" gate="G$1" x="276.86" y="147.32" smashed="yes">
+<attribute name="NAME" x="298.45" y="154.94" size="1.778" layer="95" align="center-left"/>
+<attribute name="VALUE" x="298.45" y="152.4" size="1.778" layer="96" align="center-left"/>
 </instance>
 </instances>
@@
 <label x="187.96" y="177.8" size="1.778" layer="95"/>
 </segment>
+<segment>
+<pinref part="S1" gate="G$1" pin="N.C._1"/>
+<wire x1="236.22" y1="-43.18" x2="233.68" y2="-43.18" width="0.1524" layer="91"/>
+<label x="233.68" y="-43.18" size="1.778" layer="95" rot="R180"/>
+</segment>
 </net>
 <net name="GND" class="0">
@@
 <label x="154.94" y="154.94" size="1.778" layer="95" rot="R180"/>
 </segment>
+<segment>
+<pinref part="S1" gate="G$1" pin="N.O._1"/>
+<wire x1="236.22" y1="-48.26" x2="233.68" y2="-48.26" width="0.1524" layer="91"/>
+<label x="233.68" y="-48.26" size="1.778" layer="95" rot="R180"/>
+</segment>
 </net>
 <net name="DIP0" class="0">
@@
 <wire x1="198.12" y1="-10.16" x2="198.12" y2="-43.18" width="0.1524" layer="91"/>
 <wire x1="198.12" y1="-43.18" x2="226.06" y2="-43.18" width="0.1524" layer="91"/>
-</segment>
-</net>
+<wire x1="226.06" y1="-43.18" x2="226.06" y2="-45.72" width="0.1524" layer="91"/>
+<pinref part="S1" gate="G$1" pin="COM_1"/>
+<wire x1="226.06" y1="-45.72" x2="236.22" y2="-45.72" width="0.1524" layer="91"/>
+</segment>
+</net>

Commit message: finished most boards
Parts:
- removed IC1: SN74HC02N, SamacSys_Parts:SN74HC02N
- added C1, C2, C3, C4: (no value), rcl:C-US025-024X044
- added LED0, LED1, LED10, LED11, LED12, LED13, LED14, LED15, LED2, LED3, LED4, LED5, LED6, LED7, LED8, LED9: RED, led:LED3MM
- added R0, R1, R10, R11, R12, R13, R14, R15, R2, R3, R4, R5, R6, R7, R8, R9: 220, rcl:R-US_0204/7
Connections:
- new net N$10: LED8.A, R8.1
- new net N$11: LED9.A, R9.1
- new net N$12: LED10.A, R10.1
- new net N$13: LED11.A, R11.1
- new net N$14: LED12.A, R12.1
- new net N$15: LED13.A, R13.1
- new net N$16: LED14.A, R14.1
- new net N$17: LED15.A, R15.1
- new net N$18: LED0.A, R0.1
- new net N$4: LED2.A, R2.1
- new net N$5: LED3.A, R3.1
- new net N$6: LED4.A, R4.1
- new net N$7: LED5.A, R5.1
- new net N$8: LED6.A, R6.1
- new net N$9: LED7.A, R7.1
- net GND: now also ARDUINO_WRITE.1Y, C1.1, C2.1, C3.1, C4.1, MEMORY_0-7.WE#, MEMORY_8-15.WE#
- net N$1: now also LED1.A, R1.1; no longer ARDUINO_WRITE.1Y, MEMORY_0-7.WE#, MEMORY_8-15.WE#
- net RAM0: now also R0.2
- net RAM1: now also R1.2
- net RAM10: now also R10.2
- net RAM11: now also R11.2
- net RAM12: now also R12.2
- net RAM13: now also R13.2
- net RAM14: now also R14.2
- net RAM15: now also R15.2
- net RAM2: now also R2.2
- net RAM3: now also R3.2
- net RAM4: now also R4.2
- net RAM5: now also R5.2
- net RAM6: now also R6.2
- net RAM7: now also R7.2
- net RAM8: now also R8.2
- net RAM9: now also R9.2
- net VCC: now also C1.2, C2.2, C3.2, C4.2

Commit message: added gerber files for ordering boards
Connections:
- net GND: now also LED0.C, LED1.C, LED10.C, LED11.C, LED12.C, LED13.C, LED14.C, LED15.C, LED2.C, LED3.C, LED4.C, LED5.C, LED6.C, LED7.C, LED8.C, LED9.C
Changed lines of the file:
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@@
 <wire x1="86.36" y1="147.32" x2="86.36" y2="144.78" width="0.1524" layer="91"/>
 <junction x="86.36" y="144.78"/>
+<wire x1="182.88" y1="147.32" x2="185.42" y2="147.32" width="0.1524" layer="91"/>
+<junction x="182.88" y="147.32"/>
+<label x="185.42" y="147.32" size="1.778" layer="95"/>
 </segment>
 <segment>
@@
 <junction x="297.18" y="137.16"/>
 </segment>
+<segment>
+<pinref part="LED15" gate="G$1" pin="C"/>
+<wire x1="132.08" y1="-129.54" x2="132.08" y2="-137.16" width="0.1524" layer="91"/>
+<wire x1="132.08" y1="-137.16" x2="142.24" y2="-137.16" width="0.1524" layer="91"/>
+<pinref part="LED0" gate="G$1" pin="C"/>
+<wire x1="142.24" y1="-137.16" x2="152.4" y2="-137.16" width="0.1524" layer="91"/>
+<wire x1="152.4" y1="-137.16" x2="162.56" y2="-137.16" width="0.1524" layer="91"/>
+<wire x1="162.56" y1="-137.16" x2="172.72" y2="-137.16" width="0.1524" layer="91"/>
+<wire x1="172.72" y1="-137.16" x2="182.88" y2="-137.16" width="0.1524" layer="91"/>
+<wire x1="182.88" y1="-137.16" x2="193.04" y2="-137.16" width="0.1524" layer="91"/>
+<wire x1="193.04" y1="-137.16" x2="203.2" y2="-137.16" width="0.1524" layer="91"/>
+<wire x1="203.2" y1="-137.16" x2="213.36" y2="-137.16" width="0.1524" layer="91"/>
+<wire x1="213.36" y1="-137.16" x2="223.52" y2="-137.16" width="0.1524" layer="91"/>
+<wire x1="223.52" y1="-137.16" x2="233.68" y2="-137.16" width="0.1524" layer="91"/>
+<wire x1="233.68" y1="-137.16" x2="243.84" y2="-137.16" width="0.1524" layer="91"/>
+<wire x1="243.84" y1="-137.16" x2="254" y2="-137.16" width="0.1524" layer="91"/>
+<wire x1="254" y1="-137.16" x2="264.16" y2="-137.16" width="0.1524" layer="91"/>
+<wire x1="264.16" y1="-137.16" x2="274.32" y2="-137.16" width="0.1524" layer="91"/>
+<wire x1="274.32" y1="-137.16" x2="284.48" y2="-137.16" width="0.1524" layer="91"/>
+<wire x1="287.02" y1="-137.16" x2="284.48" y2="-137.16" width="0.1524" layer="91"/>
+<wire x1="284.48" y1="-137.16" x2="284.48" y2="-129.54" width="0.1524" layer="91"/>
+<label x="287.02" y="-137.16" size="1.778" layer="95"/>
+<pinref part="LED14" gate="G$1" pin="C"/>
+<wire x1="142.24" y1="-129.54" x2="142.24" y2="-137.16" width="0.1524" layer="91"/>
+<junction x="142.24" y="-137.16"/>
+<pinref part="LED13" gate="G$1" pin="C"/>
+<wire x1="152.4" y1="-129.54" x2="152.4" y2="-137.16" width="0.1524" layer="91"/>
+<junction x="152.4" y="-137.16"/>
+<pinref part="LED12" gate="G$1" pin="C"/>
+<wire x1="162.56" y1="-129.54" x2="162.56" y2="-137.16" width="0.1524" layer="91"/>
+<junction x="162.56" y="-137.16"/>
+<pinref part="LED11" gate="G$1" pin="C"/>
+<wire x1="172.72" y1="-129.54" x2="172.72" y2="-137.16" width="0.1524" layer="91"/>
+<junction x="172.72" y="-137.16"/>
+<pinref part="LED10" gate="G$1" pin="C"/>
+<wire x1="182.88" y1="-129.54" x2="182.88" y2="-137.16" width="0.1524" layer="91"/>
+<junction x="182.88" y="-137.16"/>
+<pinref part="LED9" gate="G$1" pin="C"/>
+<wire x1="193.04" y1="-129.54" x2="193.04" y2="-137.16" width="0.1524" layer="91"/>
+<junction x="193.04" y="-137.16"/>
+<pinref part="LED8" gate="G$1" pin="C"/>
+<wire x1="203.2" y1="-129.54" x2="203.2" y2="-137.16" width="0.1524" layer="91"/>
+<junction x="203.2" y="-137.16"/>
+<pinref part="LED7" gate="G$1" pin="C"/>
+<wire x1="213.36" y1="-129.54" x2="213.36" y2="-137.16" width="0.1524" layer="91"/>
+<junction x="213.36" y="-137.16"/>
+<pinref part="LED1" gate="G$1" pin="C"/>
+<wire x1="274.32" y1="-129.54" x2="274.32" y2="-137.16" width="0.1524" layer="91"/>
+<junction x="274.32" y="-137.16"/>
+<pinref part="LED2" gate="G$1" pin="C"/>
+<wire x1="264.16" y1="-129.54" x2="264.16" y2="-137.16" width="0.1524" layer="91"/>
+<junction x="264.16" y="-137.16"/>
+<pinref part="LED3" gate="G$1" pin="C"/>
+<wire x1="254" y1="-129.54" x2="254" y2="-137.16" width="0.1524" layer="91"/>
+<junction x="254" y="-137.16"/>
+<pinref part="LED4" gate="G$1" pin="C"/>
+<wire x1="243.84" y1="-129.54" x2="243.84" y2="-137.16" width="0.1524" layer="91"/>
+<junction x="243.84" y="-137.16"/>
+<pinref part="LED5" gate="G$1" pin="C"/>
+<wire x1="233.68" y1="-129.54" x2="233.68" y2="-137.16" width="0.1524" layer="91"/>
+<junction x="233.68" y="-137.16"/>
+<pinref part="LED6" gate="G$1" pin="C"/>
+<wire x1="223.52" y1="-129.54" x2="223.52" y2="-137.16" width="0.1524" layer="91"/>
+<junction x="223.52" y="-137.16"/>
+</segment>
 </net>
