File: Eagle/Memory/memory_mkII.sch (EAGLE design)
At the start: 55 parts

Commit message: started adding revision 2 to fix errors in first set of boards
Parts:
- removed ACC=0_0-7, ACC=0_8-15: CD4048BE, SamacSys_Parts:CD4048BE
- removed ACCUMULATOR_0-7, ACCUMULATOR_8-15: SN74BCT374N, SamacSys_Parts:SN74BCT374N
- removed ACO_0-7, ACO_8-15, SKIPCOND: SN74HC541N, SamacSys_Parts:SN74HC541N
- removed ALU: 55959-1630, SamacSys_Parts:55959-1630
- removed NOT_GATE: SN74HC04N, SamacSys_Parts:SN74HC04N
- removed OR_GATE: SN74HC32N, SamacSys_Parts:SN74HC32N
- removed RSC_000, RSC_400, RSC_800: (no value), rcl:R-US_0204/7
- removed SC_000, SC_400, SC_800: (no value), led:LED3MM
- removed TRIPLE_AND_GATE: SN74HC11N, SamacSys_Parts:SN74HC11N
- added ARD/BRD_0-3, ARD/BRD_12-15, ARD/BRD_4-7, ARD/BRD_8-11, ARDUINO_WRITE, BOARD_WRITE, BUS/DIP_0-3, BUS/DIP_12-15, BUS/DIP_4-7, BUS/DIP_8-11: SN74HC157N, SamacSys_Parts:SN74HC157N
- added ARDUINO: 55959-1830, SamacSys_Parts:55959-1830
- added DIP_0-7, DIP_8-15: ADE08A04, SamacSys_Parts:ADE08A04
- added MAR: 55959-1430, SamacSys_Parts:55959-1430
- added MEMORY_0-7, MEMORY_8-15: AS6C6264-55PIN, SamacSys_Parts:AS6C6264-55PIN
- added RAM_OUT_0-7, RAM_OUT_8-15: SN74HC541N, SamacSys_Parts:SN74HC541N
- added S1: MHPS2273N, SamacSys_Parts:MHPS2273N
- LED0, LED1, LED10, LED11, LED12, LED13, LED14, LED15, LED2, LED3, LED4, LED5, LED6, LED7, LED8, LED9: value (none) -> RED
- R0, R1, R10, R11, R12, R13, R14, R15, R2, R3, R4, R5, R6, R7, R8, R9: value (none) -> 220
Connections:
- removed net AC0: ACC=0_0-7.A, ACCUMULATOR_0-7.1Q, ACO_0-7.A1, ALU.1, R0.2
- removed net AC1: ACC=0_0-7.B, ACCUMULATOR_0-7.2Q, ACO_0-7.A2, ALU.3, R1.2
- removed net AC10: ACC=0_8-15.C, ACCUMULATOR_8-15.3Q, ACO_8-15.A3, ALU.6, R10.2
- removed net AC11: ACC=0_8-15.D, ACCUMULATOR_8-15.4Q, ACO_8-15.A4, ALU.8, R11.2
- removed net AC12: ACC=0_8-15.E, ACCUMULATOR_8-15.5Q, ACO_8-15.A5, ALU.10, R12.2
- removed net AC13: ACC=0_8-15.F, ACCUMULATOR_8-15.6Q, ACO_8-15.A6, ALU.12, R13.2
- removed net AC14: ACC=0_8-15.G, ACCUMULATOR_8-15.7Q, ACO_8-15.A7, ALU.14, R14.2
- removed net AC15: ACC=0_8-15.H, ACCUMULATOR_8-15.8Q, ACO_8-15.A8, ALU.16, NOT_GATE.1A, R15.2, TRIPLE_AND_GATE.1C
- removed net AC2: ACC=0_0-7.C, ACCUMULATOR_0-7.3Q, ACO_0-7.A3, ALU.5, R2.2
- removed net AC3: ACC=0_0-7.D, ACCUMULATOR_0-7.4Q, ACO_0-7.A4, ALU.7, R3.2
- removed net AC4: ACC=0_0-7.E, ACCUMULATOR_0-7.5Q, ACO_0-7.A5, ALU.9, R4.2
- removed net AC5: ACC=0_0-7.F, ACCUMULATOR_0-7.6Q, ACO_0-7.A6, ALU.11, R5.2
- removed net AC6: ACC=0_0-7.G, ACCUMULATOR_0-7.7Q, ACO_0-7.A7, ALU.13, R6.2
- removed net AC7: ACC=0_0-7.H, ACCUMULATOR_0-7.8Q, ACO_0-7.A8, ALU.15, R7.2
- removed net AC8: ACC=0_8-15.A, ACCUMULATOR_8-15.1Q, ACO_8-15.A1, ALU.2, R8.2
- removed net AC9: ACC=0_8-15.B, ACCUMULATOR_8-15.2Q, ACO_8-15.A2, ALU.4, R9.2
- removed net ACI: AND_GATE.2A, BUS.17
- removed net ACO: ACO_0-7.!OE1, ACO_0-7.!OE2, ACO_8-15.!OE1, ACO_8-15.!OE2, BUS.18
- removed net CE: BUS.22, OR_GATE.2Y
- removed net N$1 (its old number): ACC=0_0-7.J, ACC=0_8-15.EXPAND
- removed net N$10 (its old number): RSC_000.2, SC_000.A
- removed net N$11 (its old number): LED0.C, LED1.C, LED10.C, LED11.C, LED12.C, LED13.C, LED14.C, LED15.C, LED2.C, LED3.C, LED4.C, LED5.C, LED6.C, LED7.C, LED8.C, LED9.C
- removed net N$12 (its old number): NOT_GATE.4Y, TRIPLE_AND_GATE.3A
- removed net N$13 (its old number): NOT_GATE.1Y, TRIPLE_AND_GATE.3B
- removed net N$15 (its old number): AND_GATE.1A, TRIPLE_AND_GATE.3Y
- removed net N$17 (its old number): AND_GATE.1Y, RSC_800.1, SKIPCOND.A3
- removed net N$32: OR_GATE.1A, SKIPCOND.Y1
- removed net N$33: OR_GATE.1B, SKIPCOND.Y2
- removed net N$34: OR_GATE.1Y, OR_GATE.2A
- removed net N$35: OR_GATE.2B, SKIPCOND.Y3
- removed net N$4 (its old number): NOT_GATE.2Y, TRIPLE_AND_GATE.1A, TRIPLE_AND_GATE.3C
- removed net N$5 (its old number): ACCUMULATOR_0-7.CLK, ACCUMULATOR_8-15.CLK, AND_GATE.2Y
- removed net N$6 (its old number): ACC=0_8-15.J, NOT_GATE.4A, TRIPLE_AND_GATE.2A
- removed net N$7 (its old number): NOT_GATE.3Y, TRIPLE_AND_GATE.1B, TRIPLE_AND_GATE.2C
- removed net N$8 (its old number): RSC_400.1, SKIPCOND.A2, TRIPLE_AND_GATE.2Y
- removed net N$9 (its old number): RSC_000.1, SKIPCOND.A1, TRIPLE_AND_GATE.1Y
- removed net SC: BUS.21, SKIPCOND.!OE1, SKIPCOND.!OE2
- new net A0: MAR.1, MEMORY_0-7.A0, MEMORY_8-15.A0
- new net A1: MAR.2, MEMORY_0-7.A1, MEMORY_8-15.A1
- new net A10: MAR.12, MEMORY_0-7.A10, MEMORY_8-15.A10
- new net A11: MAR.13, MEMORY_0-7.A11, MEMORY_8-15.A11
- new net A2: MAR.3, MEMORY_0-7.A2, MEMORY_8-15.A2
- new net A3: MAR.4, MEMORY_0-7.A3, MEMORY_8-15.A3
- new net A4: MAR.5, MEMORY_0-7.A4, MEMORY_8-15.A4
- new net A5: MAR.6, MEMORY_0-7.A5, MEMORY_8-15.A5
- new net A6: MAR.8, MEMORY_0-7.A6, MEMORY_8-15.A6
- new net A7: MAR.9, MEMORY_0-7.A7, MEMORY_8-15.A7
- new net A8: MAR.10, MEMORY_0-7.A8, MEMORY_8-15.A8
- new net A9: MAR.11, MEMORY_0-7.A9, MEMORY_8-15.A9
- new net ARD0: ARD/BRD_0-3.1B, ARDUINO.1
- new net ARD1: ARD/BRD_0-3.2B, ARDUINO.3
- new net ARD10: ARD/BRD_8-11.3B, ARDUINO.6
- new net ARD11: ARD/BRD_8-11.4B, ARDUINO.8
- new net ARD12: ARD/BRD_12-15.1B, ARDUINO.10
- new net ARD13: ARD/BRD_12-15.2B, ARDUINO.12
- new net ARD14: ARD/BRD_12-15.3B, ARDUINO.14
- new net ARD15: ARD/BRD_12-15.4B, ARDUINO.16
- new net ARD2: ARD/BRD_0-3.3B, ARDUINO.5
- new net ARD3: ARD/BRD_0-3.4B, ARDUINO.7
- new net ARD4: ARD/BRD_4-7.1B, ARDUINO.9
- new net ARD5: ARD/BRD_4-7.2B, ARDUINO.11
- new net ARD6: ARD/BRD_4-7.3B, ARDUINO.13
- new net ARD7: ARD/BRD_4-7.4B, ARDUINO.15
- new net ARD8: ARD/BRD_8-11.1B, ARDUINO.2
- new net ARD9: ARD/BRD_8-11.2B, ARDUINO.4
- new net ARDPRGM: AND_GATE.1B, ARDUINO.18, ARDUINO_WRITE.!A!/B
- new net ARDWRITE: ARDUINO.17, ARDUINO_WRITE.1B
- new net BRD0: ARD/BRD_0-3.1A, BUS/DIP_0-3.1Y
- new net BRD1: ARD/BRD_0-3.2A, BUS/DIP_0-3.2Y
- new net BRD10: ARD/BRD_8-11.3A, BUS/DIP_8-11.3Y
- new net BRD11: ARD/BRD_8-11.4A, BUS/DIP_8-11.4Y
- new net BRD12: ARD/BRD_12-15.1A, BUS/DIP_12-15.1Y
- new net BRD13: ARD/BRD_12-15.2A, BUS/DIP_12-15.2Y
- new net BRD14: ARD/BRD_12-15.3A, BUS/DIP_12-15.3Y
- new net BRD15: ARD/BRD_12-15.4A, BUS/DIP_12-15.4Y
- new net BRD2: ARD/BRD_0-3.3A, BUS/DIP_0-3.3Y
- new net BRD3: ARD/BRD_0-3.4A, BUS/DIP_0-3.4Y
- new net BRD4: ARD/BRD_4-7.1A, BUS/DIP_4-7.1Y
- new net BRD5: ARD/BRD_4-7.2A, BUS/DIP_4-7.2Y
- new net BRD6: ARD/BRD_4-7.3A, BUS/DIP_4-7.3Y
- new net BRD7: ARD/BRD_4-7.4A, BUS/DIP_4-7.4Y
- new net BRD8: ARD/BRD_8-11.1A, BUS/DIP_8-11.1Y
- new net BRD9: ARD/BRD_8-11.2A, BUS/DIP_8-11.2Y
- new net DIP0: BUS/DIP_0-3.1B, DIP_0-7.9
- new net DIP1: BUS/DIP_0-3.2B, DIP_0-7.10
- new net DIP10: BUS/DIP_8-11.3B, DIP_8-15.11
- new net DIP11: BUS/DIP_8-11.4B, DIP_8-15.12
- new net DIP12: BUS/DIP_12-15.1B, DIP_8-15.13
- new net DIP13: BUS/DIP_12-15.2B, DIP_8-15.14
- new net DIP14: BUS/DIP_12-15.3B, DIP_8-15.15
- new net DIP15: BUS/DIP_12-15.4B, DIP_8-15.16
- new net DIP2: BUS/DIP_0-3.3B, DIP_0-7.11
- new net DIP3: BUS/DIP_0-3.4B, DIP_0-7.12
- new net DIP4: BUS/DIP_4-7.1B, DIP_0-7.13
- new net DIP5: BUS/DIP_4-7.2B, DIP_0-7.14
- new net DIP6: BUS/DIP_4-7.3B, DIP_0-7.15
- new net DIP7: BUS/DIP_4-7.4B, DIP_0-7.16
- new net DIP8: BUS/DIP_8-11.1B, DIP_8-15.9
- new net DIP9: BUS/DIP_8-11.2B, DIP_8-15.10
- new net PRGM: AND_GATE.1A, BOARD_WRITE.!A!/B, BUS/DIP_0-3.!A!/B, BUS/DIP_12-15.!A!/B, BUS/DIP_4-7.!A!/B, BUS/DIP_8-11.!A!/B, MAR.7
- new net RAM0: ARD/BRD_0-3.1Y, MEMORY_0-7.DQ0, R0.2, RAM_OUT_0-7.A1
- new net RAM1: ARD/BRD_0-3.2Y, MEMORY_0-7.DQ1, R1.2, RAM_OUT_0-7.A2
- new net RAM10: ARD/BRD_8-11.3Y, MEMORY_8-15.DQ2, R10.2, RAM_OUT_8-15.A3
- new net RAM11: ARD/BRD_8-11.4Y, MEMORY_8-15.DQ3, R11.2, RAM_OUT_8-15.A4
- new net RAM12: ARD/BRD_12-15.1Y, MEMORY_8-15.DQ4, R12.2, RAM_OUT_8-15.A5
- new net RAM13: ARD/BRD_12-15.2Y, MEMORY_8-15.DQ5, R13.2, RAM_OUT_8-15.A6
- new net RAM14: ARD/BRD_12-15.3Y, MEMORY_8-15.DQ6, R14.2, RAM_OUT_8-15.A7
- new net RAM15: ARD/BRD_12-15.4Y, MEMORY_8-15.DQ7, R15.2, RAM_OUT_8-15.A8
- new net RAM2: ARD/BRD_0-3.3Y, MEMORY_0-7.DQ2, R2.2, RAM_OUT_0-7.A3
- new net RAM3: ARD/BRD_0-3.4Y, MEMORY_0-7.DQ3, R3.2, RAM_OUT_0-7.A4
- new net RAM4: ARD/BRD_4-7.1Y, MEMORY_0-7.DQ4, R4.2, RAM_OUT_0-7.A5
- new net RAM5: ARD/BRD_4-7.2Y, MEMORY_0-7.DQ5, R5.2, RAM_OUT_0-7.A6
- new net RAM6: ARD/BRD_4-7.3Y, MEMORY_0-7.DQ6, R6.2, RAM_OUT_0-7.A7
- new net RAM7: ARD/BRD_4-7.4Y, MEMORY_0-7.DQ7, R7.2, RAM_OUT_0-7.A8
- new net RAM8: ARD/BRD_8-11.1Y, MEMORY_8-15.DQ0, R8.2, RAM_OUT_8-15.A1
- new net RAM9: ARD/BRD_8-11.2Y, MEMORY_8-15.DQ1, R9.2, RAM_OUT_8-15.A2
- new net RAMCLK: AND_GATE.2Y, BOARD_WRITE.1A
- new net RAMPROG: AND_GATE.1Y, ARD/BRD_0-3.!A!/B, ARD/BRD_12-15.!A!/B, ARD/BRD_4-7.!A!/B, ARD/BRD_8-11.!A!/B
- new net RI: AND_GATE.2B, BUS.18
- new net RO: BUS.17, MEMORY_0-7.OE#, MEMORY_8-15.OE#, RAM_OUT_0-7.!OE1, RAM_OUT_0-7.!OE2, RAM_OUT_8-15.!OE1, RAM_OUT_8-15.!OE2
- new net WE: ARDUINO_WRITE.1Y, MEMORY_0-7.WE#, MEMORY_8-15.WE#
- net B0: now also BUS/DIP_0-3.1A, RAM_OUT_0-7.Y1; no longer ACCUMULATOR_0-7.1D, ACO_0-7.Y1
- net B1: now also BUS/DIP_0-3.2A, RAM_OUT_0-7.Y2; no longer ACCUMULATOR_0-7.2D, ACO_0-7.Y2
- net B10: now also BUS/DIP_8-11.3A, RAM_OUT_8-15.Y3; no longer ACCUMULATOR_8-15.3D, ACO_8-15.Y3, NOT_GATE.2A, TRIPLE_AND_GATE.2B
- net B11: now also BUS/DIP_8-11.4A, RAM_OUT_8-15.Y4; no longer ACCUMULATOR_8-15.4D, ACO_8-15.Y4, AND_GATE.1B, NOT_GATE.3A
- net B12: now also BUS/DIP_12-15.1A, RAM_OUT_8-15.Y5; no longer ACCUMULATOR_8-15.5D, ACO_8-15.Y5
- net B13: now also BUS/DIP_12-15.2A, RAM_OUT_8-15.Y6; no longer ACCUMULATOR_8-15.6D, ACO_8-15.Y6
- net B14: now also BUS/DIP_12-15.3A, RAM_OUT_8-15.Y7; no longer ACCUMULATOR_8-15.7D, ACO_8-15.Y7
- net B15: now also BUS/DIP_12-15.4A, RAM_OUT_8-15.Y8; no longer ACCUMULATOR_8-15.8D, ACO_8-15.Y8
- net B2: now also BUS/DIP_0-3.3A, RAM_OUT_0-7.Y3; no longer ACCUMULATOR_0-7.3D, ACO_0-7.Y3
- net B3: now also BUS/DIP_0-3.4A, RAM_OUT_0-7.Y4; no longer ACCUMULATOR_0-7.4D, ACO_0-7.Y4
- net B4: now also BUS/DIP_4-7.1A, RAM_OUT_0-7.Y5; no longer ACCUMULATOR_0-7.5D, ACO_0-7.Y5
- net B5: now also BUS/DIP_4-7.2A, RAM_OUT_0-7.Y6; no longer ACCUMULATOR_0-7.6D, ACO_0-7.Y6
- net B6: now also BUS/DIP_4-7.3A, RAM_OUT_0-7.Y7; no longer ACCUMULATOR_0-7.7D, ACO_0-7.Y7
- net B7: now also BUS/DIP_4-7.4A, RAM_OUT_0-7.Y8; no longer ACCUMULATOR_0-7.8D, ACO_0-7.Y8
- net B8: now also BUS/DIP_8-11.1A, RAM_OUT_8-15.Y1; no longer ACCUMULATOR_8-15.1D, ACO_8-15.Y1
- net B9: now also BUS/DIP_8-11.2A, RAM_OUT_8-15.Y2; no longer ACCUMULATOR_8-15.2D, ACO_8-15.Y2
- net CLK: now also AND_GATE.2A, BUS.21; no longer AND_GATE.2B, BUS.23
- net GND: now also ARD/BRD_0-3.!G, ARD/BRD_0-3.GND, ARD/BRD_12-15.!G, ARD/BRD_12-15.GND, ARD/BRD_4-7.!G, ARD/BRD_4-7.GND, ARD/BRD_8-11.!G, ARD/BRD_8-11.GND, ARDUINO_WRITE.!G, ARDUINO_WRITE.2A, ARDUINO_WRITE.2B, ARDUINO_WRITE.3A, ARDUINO_WRITE.3B, ARDUINO_WRITE.4A, ARDUINO_WRITE.4B, ARDUINO_WRITE.GND, BOARD_WRITE.!G, BOARD_WRITE.2A, BOARD_WRITE.2B, BOARD_WRITE.3A, BOARD_WRITE.3B, BOARD_WRITE.4A, BOARD_WRITE.4B, BOARD_WRITE.GND, BUS/DIP_0-3.!G, BUS/DIP_0-3.GND, BUS/DIP_12-15.!G, BUS/DIP_12-15.GND, BUS/DIP_4-7.!G, BUS/DIP_4-7.GND, BUS/DIP_8-11.!G, BUS/DIP_8-11.GND, LED0.C, LED1.C, LED10.C, LED11.C, LED12.C, LED13.C, LED14.C, LED15.C, LED2.C, LED3.C, LED4.C, LED5.C, LED6.C, LED7.C, LED8.C, LED9.C, MEMORY_0-7.A12, MEMORY_0-7.CE#, MEMORY_0-7.VSS, MEMORY_8-15.A12, MEMORY_8-15.CE#, MEMORY_8-15.VSS, RAM_OUT_0-7.GND, RAM_OUT_8-15.GND, S1.N.O._1; no longer ACC=0_0-7.EXPAND, ACC=0_0-7.KA, ACC=0_0-7.KB, ACC=0_0-7.KC, ACC=0_0-7.VSS, ACC=0_8-15.KA, ACC=0_8-15.KB, ACC=0_8-15.KC, ACC=0_8-15.VSS, ACCUMULATOR_0-7.GND, ACCUMULATOR_0-7.~OE, ACCUMULATOR_8-15.GND, ACCUMULATOR_8-15.~OE, ACO_0-7.GND, ACO_8-15.GND, NOT_GATE.5A, NOT_GATE.6A, NOT_GATE.GND, OR_GATE.3A, OR_GATE.3B, OR_GATE.4A, OR_GATE.4B, OR_GATE.GND, SC_000.C, SC_400.C, SC_800.C, SKIPCOND.A4, SKIPCOND.A5, SKIPCOND.A6, SKIPCOND.A7, SKIPCOND.A8, SKIPCOND.GND, TRIPLE_AND_GATE.GND
- net N$2: now also BOARD_WRITE.1B, S1.COM_1; no longer RSC_800.2, SC_800.A
- net N$3: now also ARDUINO_WRITE.1A, BOARD_WRITE.1Y; no longer RSC_400.2, SC_400.A
- net VCC: now also ARD/BRD_0-3.VCC, ARD/BRD_12-15.VCC, ARD/BRD_4-7.VCC, ARD/BRD_8-11.VCC, ARDUINO_WRITE.VCC, BOARD_WRITE.VCC, BUS/DIP_0-3.VCC, BUS/DIP_12-15.VCC, BUS/DIP_4-7.VCC, BUS/DIP_8-11.VCC, DIP_0-7.1, DIP_0-7.2, DIP_0-7.3, DIP_0-7.4, DIP_0-7.5, DIP_0-7.6, DIP_0-7.7, DIP_0-7.8, DIP_8-15.1, DIP_8-15.2, DIP_8-15.3, DIP_8-15.4, DIP_8-15.5, DIP_8-15.6, DIP_8-15.7, DIP_8-15.8, MEMORY_0-7.CE2, MEMORY_0-7.VCC, MEMORY_8-15.CE2, MEMORY_8-15.VCC, RAM_OUT_0-7.VCC, RAM_OUT_8-15.VCC, S1.N.C._1; no longer ACC=0_0-7.KD, ACC=0_0-7.VDD, ACC=0_8-15.KD, ACC=0_8-15.VDD, ACCUMULATOR_0-7.VCC, ACCUMULATOR_8-15.VCC, ACO_0-7.VCC, ACO_8-15.VCC, NOT_GATE.VCC, OR_GATE.VCC, SKIPCOND.VCC, TRIPLE_AND_GATE.VCC
Other:
- moved on the sheet: AND_GATE, BUS, C1, C2, C3, C4, LED0, LED1, LED10, LED11, LED12, LED13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
